File: Hardware/feng.kicad_pcb (KiCad board)
At the start: 2 copper layers, 91.6 x 56.5 mm, 44 parts, among them J1 PL CE CLK, J2 DATA_OUTPUT, J3 debug, J4 CONN_02, SW1 SW_SPST, SW10 SW_SPST, SW11 SW_SPST, SW12 SW_SPST, SW13 SW_SPST, SW14 SW_SPST, SW15 SW_SPST, SW16 SW_SPST, SW17 SW_SPST, SW18 SW_SPST, SW19 SW_SPST, SW2 SW_SPST, SW20 SW_SPST, SW21 SW_SPST, SW22 SW_SPST, SW23 SW_SPST, SW24 SW_SPST, SW3 SW_SPST, SW4 SW_SPST, SW5 SW_SPST, SW6 SW_SPST, SW7 SW_SPST, SW8 SW_SPST, SW9 SW_SPST, U1 74HC165D, U2 74HC165D, U3 74HC165D, U4 AMS1117-3.3

Commit message: pcb_50%
Parts:
- removed J3: debug, Connectors:1X03
- removed J4: CONN_02, Connectors:1X02
- added C5: 0.1uf, Capacitors:0805, F.Cu at (-61.5, 248.9)
- added C6: 0.1uf, Capacitors:0805, F.Cu at (-65.5, 248.9)
- added C7: 0.1uf, Capacitors:0805, F.Cu at (-69.6, 248.9)
- added C8: 22pf, Capacitors:0805, F.Cu at (-73.6, 248.9)
- added D10: WS2812B, Hardware:LED_WS2812B_PLCC4_5.0x5.0mm_P3.2mm, F.Cu at (-1.51, 229.1)
- added D11: WS2812B, Hardware:LED_WS2812B_PLCC4_5.0x5.0mm_P3.2mm, F.Cu at (18.6, 208.9)
- added D12: WS2812B, Hardware:LED_WS2812B_PLCC4_5.0x5.0mm_P3.2mm, F.Cu at (38.8, 188.8)
- added D13: WS2812B, Hardware:LED_WS2812B_PLCC4_5.0x5.0mm_P3.2mm, F.Cu at (58.9, 168.6)
- added D14: WS2812B, Hardware:LED_WS2812B_PLCC4_5.0x5.0mm_P3.2mm, F.Cu at (90.7, 137.8)
- added D15: WS2812B, Hardware:LED_WS2812B_PLCC4_5.0x5.0mm_P3.2mm, F.Cu at (118.5, 108.2)
- added D16: WS2812B, Hardware:LED_WS2812B_PLCC4_5.0x5.0mm_P3.2mm, F.Cu at (79.1, 147.7)
- added D17: WS2812B, Hardware:LED_WS2812B_PLCC4_5.0x5.0mm_P3.2mm, F.Cu at (68.6, 156.8)
- added D18: WS2812B, Hardware:LED_WS2812B_PLCC4_5.0x5.0mm_P3.2mm, F.Cu at (48.4, 176.9)
- added D19: WS2812B, Hardware:LED_WS2812B_PLCC4_5.0x5.0mm_P3.2mm, F.Cu at (28.3, 197.1)
- added D2: WS2812B, Hardware:LED_WS2812B_PLCC4_5.0x5.0mm_P3.2mm, F.Cu at (15.3, 235.4)
- added D20: WS2812B, Hardware:LED_WS2812B_PLCC4_5.0x5.0mm_P3.2mm, F.Cu at (25.0, 216.9)
- added D21: WS2812B, Hardware:LED_WS2812B_PLCC4_5.0x5.0mm_P3.2mm, F.Cu at (55.6, 188.5)
- added D22: WS2812B, Hardware:LED_WS2812B_PLCC4_5.0x5.0mm_P3.2mm, F.Cu at (95.9, 144.6)
- added D23: WS2812B, Hardware:LED_WS2812B_PLCC4_5.0x5.0mm_P3.2mm, F.Cu at (95.9, 151.3)
- added D24: WS2812B, Hardware:LED_WS2812B_PLCC4_5.0x5.0mm_P3.2mm, F.Cu at (118.2, 128.0)
- added D25: WS2812B, Hardware:LED_WS2812B_PLCC4_5.0x5.0mm_P3.2mm, F.Cu at (85.4, 161.0)
- added D26: WS2812B, Hardware:LED_WS2812B_PLCC4_5.0x5.0mm_P3.2mm, F.Cu at (107.5, 140.3)
- added D27: WS2812B, Hardware:LED_WS2812B_PLCC4_5.0x5.0mm_P3.2mm, F.Cu at (25.0, 223.6)
- added D28: WS2812B, Hardware:LED_WS2812B_PLCC4_5.0x5.0mm_P3.2mm, F.Cu at (84.2, 167.6)
- added D29: WS2812B, Hardware:LED_WS2812B_PLCC4_5.0x5.0mm_P3.2mm, F.Cu at (75.8, 174.2)
- added D3: WS2812B, Hardware:LED_WS2812B_PLCC4_5.0x5.0mm_P3.2mm, F.Cu at (35.5, 215.3)
- added D30: WS2812B, Hardware:LED_WS2812B_PLCC4_5.0x5.0mm_P3.2mm, F.Cu at (65.3, 183.3)
- added D31: WS2812B, Hardware:LED_WS2812B_PLCC4_5.0x5.0mm_P3.2mm, F.Cu at (45.1, 203.4)
- added D32: WS2812B, Hardware:LED_WS2812B_PLCC4_5.0x5.0mm_P3.2mm, F.Cu at (15.3, 228.8)
- added D33: WS2812B, Hardware:LED_WS2812B_PLCC4_5.0x5.0mm_P3.2mm, F.Cu at (4.83, 237.1)
- added D34: WS2812B, Hardware:LED_WS2812B_PLCC4_5.0x5.0mm_P3.2mm, F.Cu at (35.5, 208.6)
- added D35: WS2812B, Hardware:LED_WS2812B_PLCC4_5.0x5.0mm_P3.2mm, F.Cu at (45.1, 196.8)
- added D36: WS2812B, Hardware:LED_WS2812B_PLCC4_5.0x5.0mm_P3.2mm, F.Cu at (65.3, 176.6)
- added D37: WS2812B, Hardware:LED_WS2812B_PLCC4_5.0x5.0mm_P3.2mm, F.Cu at (3.60, 243.7)
- added D38: WS2812B, Hardware:LED_WS2812B_PLCC4_5.0x5.0mm_P3.2mm, F.Cu at (75.8, 167.6)
- added D39: WS2812B, Hardware:LED_WS2812B_PLCC4_5.0x5.0mm_P3.2mm, F.Cu at (107.5, 133.7)
- added D4: WS2812B, Hardware:LED_WS2812B_PLCC4_5.0x5.0mm_P3.2mm, F.Cu at (93.8, 157.9)
- added D40: WS2812B, Hardware:LED_WS2812B_PLCC4_5.0x5.0mm_P3.2mm, F.Cu at (104.3, 146.9)
- added D41: WS2812B, Hardware:LED_WS2812B_PLCC4_5.0x5.0mm_P3.2mm, F.Cu at (55.6, 195.1)
- added D42: WS2812B, Hardware:LED_WS2812B_PLCC4_5.0x5.0mm_P3.2mm, F.Cu at (33.4, 221.9)
- added D43: WS2812B, Hardware:LED_WS2812B_PLCC4_5.0x5.0mm_P3.2mm, F.Cu at (73.7, 180.8)
- added D44: WS2812B, Hardware:LED_WS2812B_PLCC4_5.0x5.0mm_P3.2mm, F.Cu at (53.5, 201.7)
- added D45: WS2812B, Hardware:LED_WS2812B_PLCC4_5.0x5.0mm_P3.2mm, F.Cu at (23.7, 230.2)
- added D46: WS2812B, Hardware:LED_WS2812B_PLCC4_5.0x5.0mm_P3.2mm, F.Cu at (43.9, 210.0)
- added D47: WS2812B, Hardware:LED_WS2812B_PLCC4_5.0x5.0mm_P3.2mm, F.Cu at (64.0, 189.9)
- added D48: WS2812B, Hardware:LED_WS2812B_PLCC4_5.0x5.0mm_P3.2mm, F.Cu at (-13.2, 244.0)
- added D49: WS2812B, Hardware:LED_WS2812B_PLCC4_5.0x5.0mm_P3.2mm, F.Cu at (85.4, 154.4)
- added D5: WS2812B, Hardware:LED_WS2812B_PLCC4_5.0x5.0mm_P3.2mm, F.Cu at (68.6, 150.2)
- added D50: WS2812B, Hardware:LED_WS2812B_PLCC4_5.0x5.0mm_P3.2mm, F.Cu at (77.0, 161.0)
- added D51: WS2812B, Hardware:LED_WS2812B_PLCC4_5.0x5.0mm_P3.2mm, F.Cu at (67.4, 170.0)
- added D52: WS2812B, Hardware:LED_WS2812B_PLCC4_5.0x5.0mm_P3.2mm, F.Cu at (47.2, 190.2)
- added D53: WS2812B, Hardware:LED_WS2812B_PLCC4_5.0x5.0mm_P3.2mm, F.Cu at (27.1, 210.3)
- added D54: WS2812B, Hardware:LED_WS2812B_PLCC4_5.0x5.0mm_P3.2mm, F.Cu at (6.91, 230.5)
- added D55: WS2812B, Hardware:LED_WS2812B_PLCC4_5.0x5.0mm_P3.2mm, F.Cu at (16.6, 222.2)
- added D56: WS2812B, Hardware:LED_WS2812B_PLCC4_5.0x5.0mm_P3.2mm, F.Cu at (36.7, 202.0)
- added D57: WS2812B, Hardware:LED_WS2812B_PLCC4_5.0x5.0mm_P3.2mm, F.Cu at (56.9, 181.9)
- added D58: WS2812B, Hardware:LED_WS2812B_PLCC4_5.0x5.0mm_P3.2mm, F.Cu at (-4.82, 244.0)
- added D59: WS2812B, Hardware:LED_WS2812B_PLCC4_5.0x5.0mm_P3.2mm, F.Cu at (99.1, 138.0)
- added D6: WS2812B, Hardware:LED_WS2812B_PLCC4_5.0x5.0mm_P3.2mm, F.Cu at (48.4, 170.3)
- added D60: WS2812B, Hardware:LED_WS2812B_PLCC4_5.0x5.0mm_P3.2mm, F.Cu at (118.2, 114.8)
- added D61: WS2812B, Hardware:LED_WS2812B_PLCC4_5.0x5.0mm_P3.2mm, F.Cu at (77.0, 154.4)
- added D62: WS2812B, Hardware:LED_WS2812B_PLCC4_5.0x5.0mm_P3.2mm, F.Cu at (118.2, 121.4)
- added D63: WS2812B, Hardware:LED_WS2812B_PLCC4_5.0x5.0mm_P3.2mm, F.Cu at (67.4, 163.4)
- added D64: WS2812B, Hardware:LED_WS2812B_PLCC4_5.0x5.0mm_P3.2mm, F.Cu at (47.2, 183.5)
- added D65: WS2812B, Hardware:LED_WS2812B_PLCC4_5.0x5.0mm_P3.2mm, F.Cu at (27.1, 203.7)
- added D66: WS2812B, Hardware:LED_WS2812B_PLCC4_5.0x5.0mm_P3.2mm, F.Cu at (6.91, 223.8)
- added D67: WS2812B, Hardware:LED_WS2812B_PLCC4_5.0x5.0mm_P3.2mm, F.Cu at (16.6, 215.5)
- added D68: WS2812B, Hardware:LED_WS2812B_PLCC4_5.0x5.0mm_P3.2mm, F.Cu at (36.7, 195.4)
- added D69: WS2812B, Hardware:LED_WS2812B_PLCC4_5.0x5.0mm_P3.2mm, F.Cu at (56.9, 175.2)
- added D7: WS2812B, Hardware:LED_WS2812B_PLCC4_5.0x5.0mm_P3.2mm, F.Cu at (12.0, 243.7)
- added D70: WS2812B, Hardware:LED_WS2812B_PLCC4_5.0x5.0mm_P3.2mm, F.Cu at (87.5, 147.7)
- added D71: WS2812B, Hardware:LED_WS2812B_PLCC4_5.0x5.0mm_P3.2mm, F.Cu at (99.1, 131.4)
- added D72: WS2812B, Hardware:LED_WS2812B_PLCC4_5.0x5.0mm_P3.2mm, F.Cu at (109.7, 120.4)
- added D73: WS2812B, Hardware:LED_WS2812B_PLCC4_5.0x5.0mm_P3.2mm, F.Cu at (28.3, 190.5)
- added D74: WS2812B, Hardware:LED_WS2812B_PLCC4_5.0x5.0mm_P3.2mm, F.Cu at (-3.59, 235.7)
- added D75: WS2812B, Hardware:LED_WS2812B_PLCC4_5.0x5.0mm_P3.2mm, F.Cu at (109.7, 127.0)
- added D76: WS2812B, Hardware:LED_WS2812B_PLCC4_5.0x5.0mm_P3.2mm, F.Cu at (8.14, 217.2)
- added D77: WS2812B, Hardware:LED_WS2812B_PLCC4_5.0x5.0mm_P3.2mm, F.Cu at (-12.0, 237.4)
- added D78: WS2812B, Hardware:LED_WS2812B_PLCC4_5.0x5.0mm_P3.2mm, F.Cu at (58.9, 162.0)
- added D79: WS2812B, Hardware:LED_WS2812B_PLCC4_5.0x5.0mm_P3.2mm, F.Cu at (38.8, 182.2)
- added D8: WS2812B, Hardware:LED_WS2812B_PLCC4_5.0x5.0mm_P3.2mm, F.Cu at (109.7, 113.8)
- added D80: WS2812B, Hardware:LED_WS2812B_PLCC4_5.0x5.0mm_P3.2mm, F.Cu at (18.6, 202.3)
- added D81: WS2812B, Hardware:LED_WS2812B_PLCC4_5.0x5.0mm_P3.2mm, F.Cu at (-1.51, 222.5)
- added D82: WS2812B, Hardware:LED_WS2812B_PLCC4_5.0x5.0mm_P3.2mm, F.Cu at (118.5, 101.6)
- added D83: WS2812B, Hardware:LED_WS2812B_PLCC4_5.0x5.0mm_P3.2mm, F.Cu at (-21.7, 242.6)
- added D84: WS2812B, Hardware:LED_WS2812B_PLCC4_5.0x5.0mm_P3.2mm, F.Cu at (-12.0, 230.8)
- added D85: WS2812B, Hardware:LED_WS2812B_PLCC4_5.0x5.0mm_P3.2mm, F.Cu at (8.14, 210.6)
- added D9: WS2812B, Hardware:LED_WS2812B_PLCC4_5.0x5.0mm_P3.2mm, F.Cu at (-21.7, 249.2)
- added R1: 10K, Resistors:0805, F.Cu at (-41.3, 248.9)
- added R2: 1M, Resistors:0805, F.Cu at (-45.3, 248.9)
- added R3: 5.1K, Resistors:0805, F.Cu at (-37.2, 248.9)
- added R4: 1K, Resistors:0805, F.Cu at (124.5, 87.7)
- added R6: 22, Resistors:0805, F.Cu at (-33.2, 248.9)
- added R7: 1.5k, Resistors:0805, F.Cu at (-29.2, 248.9)
- added RN10: R_Pack04, Resistor_SMD:R_Array_Convex_4x0603, F.Cu at (-119.2, 250.0)
- added RN11: R_Pack04, Resistor_SMD:R_Array_Convex_4x0603, F.Cu at (-127.5, 250.0)
- added RN12: R_Pack04, Resistor_SMD:R_Array_Convex_4x0603, F.Cu at (-131.6, 250.0)
- added RN13: R_Pack04, Resistor_SMD:R_Array_Convex_4x0603, F.Cu at (-135.8, 250.0)
- added RN14: R_Pack04, Resistor_SMD:R_Array_Convex_4x0603, F.Cu at (-139.9, 250.0)
- added RN15: R_Pack04, Resistor_SMD:R_Array_Convex_4x0603, F.Cu at (-144.1, 250.0)
- added RN16: R_Pack04, Resistor_SMD:R_Array_Convex_4x0603, F.Cu at (-148.2, 250.0)
- added RN17: R_Pack04, Resistor_SMD:R_Array_Convex_4x0603, F.Cu at (-156.5, 250.0)
- added RN18: R_Pack04, Resistor_SMD:R_Array_Convex_4x0603, F.Cu at (-110.9, 250.0)
- added RN19: R_Pack04, Resistor_SMD:R_Array_Convex_4x0603, F.Cu at (-115.0, 250.0)
- added RN20: R_Pack04, Resistor_SMD:R_Array_Convex_4x0603, F.Cu at (-123.3, 250.0)
- added RN21: R_Pack04, Resistor_SMD:R_Array_Convex_4x0603, F.Cu at (-152.4, 250.0)
- added RN22: R_Pack04, Resistor_SMD:R_Array_Convex_4x0603, F.Cu at (-164.8, 250.0)
- added RN7: R_Pack04, Resistor_SMD:R_Array_Convex_4x0603, F.Cu at (-106.7, 250.0)
- added RN8: R_Pack04, Resistor_SMD:R_Array_Convex_4x0603, F.Cu at (-77.7, 250.0)
- added RN9: R_Pack04, Resistor_SMD:R_Array_Convex_4x0603, F.Cu at (-160.7, 250.0)
- added SW25: SW_SPST, Switch_Keyboard_Hotswap_Kailh:SW_Hotswap_Kailh_MX_1.00u, F.Cu at (314.0, 182.8)
- added SW26: SW_SPST, Switch_Keyboard_Hotswap_Kailh:SW_Hotswap_Kailh_MX_1.00u, F.Cu at (428.2, 159.0)
- added SW27: SW_SPST, Switch_Keyboard_Hotswap_Kailh:SW_Hotswap_Kailh_MX_1.00u, F.Cu at (375.9, 240.0)
- added SW28: SW_SPST, Switch_Keyboard_Hotswap_Kailh:SW_Hotswap_Kailh_MX_1.00u, F.Cu at (390.2, 259.0)
- added SW29: SW_SPST, Switch_Keyboard_Hotswap_Kailh:SW_Hotswap_Kailh_MX_1.00u, F.Cu at (323.5, 201.9)
- added SW30: SW_SPST, Switch_Keyboard_Hotswap_Kailh:SW_Hotswap_Kailh_MX_1.00u, F.Cu at (309.1, 220.9)
- added SW31: SW_SPST, Switch_Keyboard_Hotswap_Kailh:SW_Hotswap_Kailh_MX_1.00u, F.Cu at (-56.1, 177.1)
- added SW32: SW_SPST, Switch_Keyboard_Hotswap_Kailh:SW_Hotswap_Kailh_MX_1.00u, F.Cu at (-76.2, 197.2)
- added SW33: SW_SPST, Switch_Keyboard_Hotswap_Kailh:SW_Hotswap_Kailh_MX_1.00u, F.Cu at (-96.4, 217.4)
- added SW34: SW_SPST, Switch_Keyboard_Hotswap_Kailh:SW_Hotswap_Kailh_MX_1.00u, F.Cu at (490.8, 177.4)
- added SW35: SW_SPST, Switch_Keyboard_Hotswap_Kailh:SW_Hotswap_Kailh_MX_1.00u, F.Cu at (-76.2, 217.4)
- added SW36: SW_SPST, Switch_Keyboard_Hotswap_Kailh:SW_Hotswap_Kailh_MX_1.00u, F.Cu at (399.7, 201.9)
- added SW37: SW_SPST, Switch_Keyboard_Hotswap_Kailh:SW_Hotswap_Kailh_MX_1.00u, F.Cu at (347.1, 220.9)
- added SW38: SW_SPST, Switch_Keyboard_Hotswap_Kailh:SW_Hotswap_Kailh_MX_1.00u, F.Cu at (385.3, 220.9)
- added SW39: SW_SPST, Switch_Keyboard_Hotswap_Kailh:SW_Hotswap_Kailh_MX_1.00u, F.Cu at (24.5, 177.1)
- added SW40: SW_SPST, Switch_Keyboard_Hotswap_Kailh:SW_Hotswap_Kailh_MX_1.00u, F.Cu at (4.35, 197.2)
- added SW41: SW_SPST, Switch_Keyboard_Hotswap_Kailh:SW_Hotswap_Kailh_MX_1.00u, F.Cu at (-15.8, 217.4)
- added SW42: SW_SPST, Switch_Keyboard_Hotswap_Kailh:SW_Hotswap_Kailh_MX_1.00u, F.Cu at (299.7, 240.0)
- added SW43: SW_SPST, Switch_Keyboard_Hotswap_Kailh:SW_Hotswap_Kailh_MX_1.00u, F.Cu at (-116.5, 177.1)
- added SW44: SW_SPST, Switch_Keyboard_Hotswap_Kailh:SW_Hotswap_Kailh_MX_1.00u, F.Cu at (-136.7, 197.2)
- added SW45: SW_SPST, Switch_Keyboard_Hotswap_Kailh:SW_Hotswap_Kailh_MX_1.00u, F.Cu at (266.3, 201.9)
- added SW46: SW_SPST, Switch_Keyboard_Hotswap_Kailh:SW_Hotswap_Kailh_MX_1.00u, F.Cu at (275.9, 182.8)
- added SW47: SW_SPST, Switch_Keyboard_Hotswap_Kailh:SW_Hotswap_Kailh_MX_1.00u, F.Cu at (318.7, 240.0)
- added SW48: SW_SPST, Switch_Keyboard_Hotswap_Kailh:SW_Hotswap_Kailh_MX_1.00u, F.Cu at (456.8, 220.9)
- added SW49: SW_SPST, Switch_Keyboard_Hotswap_Kailh:SW_Hotswap_Kailh_MX_1.00u, F.Cu at (-136.7, 217.4)
- added SW50: SW_SPST, Switch_Keyboard_Hotswap_Kailh:SW_Hotswap_Kailh_MX_1.00u, F.Cu at (-116.5, 197.2)
- added SW51: SW_SPST, Switch_Keyboard_Hotswap_Kailh:SW_Hotswap_Kailh_MX_1.00u, F.Cu at (-96.4, 177.1)
- added SW52: SW_SPST, Switch_Keyboard_Hotswap_Kailh:SW_Hotswap_Kailh_MX_1.00u, F.Cu at (-156.8, 217.4)
- added SW53: SW_SPST, Switch_Keyboard_Hotswap_Kailh:SW_Hotswap_Kailh_MX_1.00u, F.Cu at (285.4, 201.9)
- added SW54: SW_SPST, Switch_Keyboard_Hotswap_Kailh:SW_Hotswap_Kailh_MX_1.00u, F.Cu at (295.0, 182.8)
- added SW55: SW_SPST, Switch_Keyboard_Hotswap_Kailh:SW_Hotswap_Kailh_MX_1.00u, F.Cu at (337.8, 240.0)
- added SW56: SW_SPST, Switch_Keyboard_Hotswap_Kailh:SW_Hotswap_Kailh_MX_1.00u, F.Cu at (252.0, 220.9)
- added SW57: SW_SPST, Switch_Keyboard_Hotswap_Kailh:SW_Hotswap_Kailh_MX_1.00u, F.Cu at (456.8, 201.9)
- added SW58: SW_SPST, Switch_Keyboard_Hotswap_Kailh:SW_Hotswap_Kailh_MX_1.00u, F.Cu at (356.8, 240.0)
- added SW59: SW_SPST, Switch_Keyboard_Hotswap_Kailh:SW_Hotswap_Kailh_MX_1.00u, F.Cu at (361.7, 201.9)
- added SW60: SW_SPST, Switch_Keyboard_Hotswap_Kailh:SW_Hotswap_Kailh_MX_1.00u, F.Cu at (371.2, 182.8)
- added SW61: SW_SPST, Switch_Keyboard_Hotswap_Kailh:SW_Hotswap_Kailh_MX_1.00u, F.Cu at (371.1, 259.0)
- added SW62: SW_SPST, Switch_Keyboard_Hotswap_Kailh:SW_Hotswap_Kailh_MX_1.00u, F.Cu at (456.8, 240.0)
- added SW63: SW_SPST, Switch_Keyboard_Hotswap_Kailh:SW_Hotswap_Kailh_MX_1.00u, F.Cu at (-35.9, 217.4)
- added SW64: SW_SPST, Switch_Keyboard_Hotswap_Kailh:SW_Hotswap_Kailh_MX_1.00u, F.Cu at (-15.8, 197.2)
- added SW65: SW_SPST, Switch_Keyboard_Hotswap_Kailh:SW_Hotswap_Kailh_MX_1.00u, F.Cu at (4.35, 177.1)
- added SW66: SW_SPST, Switch_Keyboard_Hotswap_Kailh:SW_Hotswap_Kailh_MX_1.00u, F.Cu at (366.2, 220.9)
- added SW67: SW_SPST, Switch_Keyboard_Hotswap_Kailh:SW_Hotswap_Kailh_MX_1.00u, F.Cu at (380.7, 201.9)
- added SW68: SW_SPST, Switch_Keyboard_Hotswap_Kailh:SW_Hotswap_Kailh_MX_1.00u, F.Cu at (390.3, 182.8)
- added SW69: SW_SPST, Switch_Keyboard_Hotswap_Kailh:SW_Hotswap_Kailh_MX_1.00u, F.Cu at (-116.5, 217.4)
- added SW70: SW_SPST, Switch_Keyboard_Hotswap_Kailh:SW_Hotswap_Kailh_MX_1.00u, F.Cu at (218.6, 182.8)
- added SW71: SW_SPST, Switch_Keyboard_Hotswap_Kailh:SW_Hotswap_Kailh_MX_1.00u, F.Cu at (209.2, 201.9)
- added SW72: SW_SPST, Switch_Keyboard_Hotswap_Kailh:SW_Hotswap_Kailh_MX_1.00u, F.Cu at (194.9, 220.9)
- added SW73: SW_SPST, Switch_Keyboard_Hotswap_Kailh:SW_Hotswap_Kailh_MX_1.00u, F.Cu at (242.5, 240.0)
- added SW74: SW_SPST, Switch_Keyboard_Hotswap_Kailh:SW_Hotswap_Kailh_MX_1.00u, F.Cu at (199.7, 182.8)
- added SW75: SW_SPST, Switch_Keyboard_Hotswap_Kailh:SW_Hotswap_Kailh_MX_1.00u, F.Cu at (190.1, 201.9)
- added SW76: SW_SPST, Switch_Keyboard_Hotswap_Kailh:SW_Hotswap_Kailh_MX_1.00u, F.Cu at (223.5, 240.0)
- added SW77: SW_SPST, Switch_Keyboard_Hotswap_Kailh:SW_Hotswap_Kailh_MX_1.00u, F.Cu at (180.6, 182.8)
- added SW78: SW_SPST, Switch_Keyboard_Hotswap_Kailh:SW_Hotswap_Kailh_MX_1.00u, F.Cu at (213.9, 220.9)
- added SW79: SW_SPST, Switch_Keyboard_Hotswap_Kailh:SW_Hotswap_Kailh_MX_1.00u, F.Cu at (304.4, 201.9)
- added SW80: SW_SPST, Switch_Keyboard_Hotswap_Kailh:SW_Hotswap_Kailh_MX_1.00u, F.Cu at (290.1, 220.9)
- added SW81: SW_SPST, Switch_Keyboard_Hotswap_Kailh:SW_Hotswap_Kailh_MX_1.00u, F.Cu at (-76.2, 177.1)
- added SW82: SW_SPST, Switch_Keyboard_Hotswap_Kailh:SW_Hotswap_Kailh_MX_1.00u, F.Cu at (-96.4, 197.2)
- added SW83: Rotary_Encoder_Switch, Hardware:keyboard-RotaryEncoder_Alps_EC12E-Switch_Vertical_H20mm_CircularMountingHoles, F.Cu at (448.5, 157.5)
- added U10: 74HC165D, Package_SO:SOP-16_4.55x10.3mm_P1.27mm, F.Cu at (99.9, 110.8)
- added U11: 74HC165D, Package_SO:SOP-16_4.55x10.3mm_P1.27mm, F.Cu at (99.9, 99.0)
- added U12: STM32F103C8Tx, Package_QFP:LQFP-48_7x7mm_P0.5mm, F.Cu at (99.9, 122.4)
- added U5: 74HC165D, Package_SO:SOP-16_4.55x10.3mm_P1.27mm, F.Cu at (39.4, 172.9)
- added U6: 74HC165D, Package_SO:SOP-16_4.55x10.3mm_P1.27mm, F.Cu at (117.7, 92.3)
- added U7: 74HC165D, Package_SO:SOP-16_4.55x10.3mm_P1.27mm, F.Cu at (-0.90, 213.2)
- added U8: 74HC165D, Package_SO:SOP-16_4.55x10.3mm_P1.27mm, F.Cu at (-21.0, 233.4)
- added U9: 74HC165D, Package_SO:SOP-16_4.55x10.3mm_P1.27mm, F.Cu at (79.7, 128.5)
- added Y1: 8M, Crystal:Crystal_HC49-4H_Vertical, F.Cu at (99.2, 89.7)
- C1: value 10UF-0805-10V-10% -> 0.1uf; moved to F.Cu
- C2: value 0.1UF-0603-25V-5% -> 22pf; moved to F.Cu
- C3: value 10UF-0805-10V-10% -> 10uf; moved to F.Cu
- C4: value 0.1UF-0603-25V-5% -> 0.1uf; moved to F.Cu
- D1: value LED -> WS2812B; footprint LED_THT:LED_D3.0mm -> Hardware:LED_WS2812B_PLCC4_5.0x5.0mm_P3.2mm
- J1: value PL CE CLK -> STLINK_PLUG; footprint Connector_PinHeader_2.54mm:PinHeader_1x03_P2.54mm_Vertical -> Connector_PinHeader_2.54mm:PinHeader_1x04_P2.54mm_Vertical
- J2: value DATA_OUTPUT -> USB_C_Receptacle_USB2.0; footprint Connectors:1X01 -> Connector_USB:USB_C_Receptacle_Palconn_UTC16-G
- R5: value 10k -> 22; footprint Resistor_THT:R_Axial_DIN0309_L9.0mm_D3.2mm_P12.70mm_Horizontal -> Resistors:0805
- RN1, RN2, RN3, RN4, RN5, RN6, U1, U2, U3: moved to F.Cu
- SW1, SW10, SW11, SW12, SW13, SW14, SW15, SW16, SW17, SW18, SW19, SW2, SW20, SW21, SW22, SW23, SW24, SW3, SW4, SW5, SW6, SW7, SW8, SW9: footprint Button_Switch_THT:SW_DIP_SPSTx01_Slide_6.7x4.1mm_W7.62mm_P2.54mm_LowProfile -> Switch_Keyboard_Hotswap_Kailh:SW_Hotswap_Kailh_MX_1.00u
- U4: value AMS1117-3.3 -> 74HC165D; footprint Package_TO_SOT_SMD:SOT-223-3_TabPin2 -> Package_SO:SOP-16_4.55x10.3mm_P1.27mm; moved to F.Cu
- moved SW1 342.6 mm to (452.0, 263.8)
- moved RN6 328.4 mm to (-102.6, 250.0), turned to 0 degrees
- moved RN3 323.2 mm to (-90.1, 250.0), turned to 0 degrees
- moved SW12 316.6 mm to (-156.8, 177.1)
- moved SW18 311.1 mm to (456.8, 182.8)
- moved RN5 307.7 mm to (-98.4, 250.0), turned to 0 degrees
- moved RN2 302.7 mm to (-86.0, 250.0), turned to 0 degrees
- moved SW7 297.4 mm to (-156.8, 197.2)
- moved RN4 287.9 mm to (-94.3, 250.0), turned to 0 degrees
- moved RN1 283.2 mm to (-81.8, 250.0), turned to 0 degrees
- moved SW6 280.4 mm to (-136.7, 177.1)
- moved C4 276.0 mm to (-57.4, 248.9), turned to 0 degrees
- moved C3 271.8 mm to (-53.4, 248.9), turned to 0 degrees
- moved SW17 268.9 mm to (-56.1, 217.4)
- moved SW19 268.7 mm to (352.0, 259.0)
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Connections:
- C1 pad 1: VDD -> Net-(C1-Pad1)
- C2 pad 1: VDD -> Net-(C2-Pad1)
- C3 pad 1: +3V3 -> GNDPWR
- C3 pad 2: GNDPWR -> +3V3
- C4 pad 1: +3V3 -> GNDPWR
- C4 pad 2: GNDPWR -> +3V3
- D1 pad 1: GNDPWR -> +3V3
- J1 pad 2: Net-(J1-Pad2) -> /SWDIO
- J1 pad 3: Net-(J1-Pad3) -> /SWCLK
- R5 pad 1: Net-(D1-Pad2) -> /USB_DN
- R5 pad 2: +3V3 -> Net-(R5-Pad2)
- SW1 pad 1: Net-(RN4-Pad4) -> Net-(RN12-Pad4)
- SW10 pad 1: Net-(RN5-Pad3) -> Net-(RN13-Pad3)
- SW11 pad 1: Net-(RN5-Pad2) -> Net-(RN13-Pad2)
- SW12 pad 1: Net-(RN5-Pad1) -> Net-(RN13-Pad1)
- SW17 pad 1: Net-(RN6-Pad4) -> Net-(RN14-Pad4)
- SW18 pad 1: Net-(RN6-Pad3) -> Net-(RN14-Pad3)
- SW19 pad 1: Net-(RN6-Pad2) -> Net-(RN14-Pad2)
- SW2 pad 1: Net-(RN4-Pad3) -> Net-(RN12-Pad3)
- SW20 pad 1: Net-(RN6-Pad1) -> Net-(RN14-Pad1)
- SW3 pad 1: Net-(RN4-Pad2) -> Net-(RN12-Pad2)
- SW4 pad 1: Net-(RN4-Pad1) -> Net-(RN12-Pad1)
- SW9 pad 1: Net-(RN5-Pad4) -> Net-(RN13-Pad4)
- U1 pad 1: Net-(J1-Pad1) -> /SCAN_PL
- U1 pad 15: Net-(J1-Pad2) -> /SCAN_CE
- U1 pad 2: Net-(J1-Pad3) -> /SPI1_CLK
- U1 pad 3: Net-(RN4-Pad1) -> Net-(RN12-Pad1)
- U1 pad 4: Net-(RN4-Pad2) -> Net-(RN12-Pad2)
- U1 pad 5: Net-(RN4-Pad3) -> Net-(RN12-Pad3)
- U1 pad 6: Net-(RN4-Pad4) -> Net-(RN12-Pad4)
- U1 pad 9: /out_1 -> /SPI1_MISO
- U2 pad 1: Net-(J1-Pad1) -> /SCAN_PL
- U2 pad 10: /out_1 -> Net-(U2-Pad10)
- U2 pad 15: Net-(J1-Pad2) -> /SCAN_CE
- U2 pad 2: Net-(J1-Pad3) -> /SPI1_CLK
- U2 pad 3: Net-(RN5-Pad1) -> Net-(RN13-Pad1)
- U2 pad 4: Net-(RN5-Pad2) -> Net-(RN13-Pad2)
- U2 pad 5: Net-(RN5-Pad3) -> Net-(RN13-Pad3)
- U2 pad 6: Net-(RN5-Pad4) -> Net-(RN13-Pad4)
- U2 pad 9: /out_2 -> Net-(U1-Pad10)
- U3 pad 1: Net-(J1-Pad1) -> /SCAN_PL
- U3 pad 10: /out_2 -> Net-(U3-Pad10)
- U3 pad 15: Net-(J1-Pad2) -> /SCAN_CE
- U3 pad 2: Net-(J1-Pad3) -> /SPI1_CLK
- U3 pad 3: Net-(RN6-Pad1) -> Net-(RN14-Pad1)
- U3 pad 4: Net-(RN6-Pad2) -> Net-(RN14-Pad2)
- U3 pad 5: Net-(RN6-Pad3) -> Net-(RN14-Pad3)
- U3 pad 6: Net-(RN6-Pad4) -> Net-(RN14-Pad4)
- U3 pad 9: /out_3 -> Net-(U2-Pad10)
- U4 pad 1: GNDPWR -> /SCAN_PL
- U4 pad 2: +3V3 -> /SPI1_CLK
- U4 pad 3: VDD -> Net-(RN15-Pad1)
Routing:
- net +3V3: track 185.4 -> 0.00 mm, vias 5 -> 0
- net Net-(RN3-Pad1): track 116.5 -> 0.00 mm, vias 2 -> 0
- net Net-(RN3-Pad2): track 104.1 -> 0.00 mm, vias 2 -> 0
- net Net-(J1-Pad1): track 94.2 -> 0.00 mm, vias 2 -> 0
- net Net-(RN2-Pad3): track 82.0 -> 0.00 mm, vias 3 -> 0
- net Net-(RN6-Pad2): track 79.4 -> 0.00 mm
- net Net-(RN6-Pad1): track 79.2 -> 0.00 mm, vias 2 -> 0
- net Net-(RN3-Pad3): track 78.4 -> 0.00 mm, vias 2 -> 0
- net Net-(RN2-Pad1): track 70.8 -> 0.00 mm, vias 2 -> 0
- net Net-(RN4-Pad4): track 68.9 -> 0.00 mm, vias 1 -> 0
- net Net-(J1-Pad2): track 66.2 -> 0.00 mm, vias 3 -> 0
- net Net-(RN3-Pad4): track 65.5 -> 0.00 mm
- net Net-(J1-Pad3): track 65.2 -> 0.00 mm, vias 3 -> 0
- net Net-(RN4-Pad2): track 64.4 -> 0.00 mm, vias 2 -> 0
- net Net-(RN4-Pad3): track 64.4 -> 0.00 mm, vias 4 -> 0
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- removed copper zone on B.Cu, net GNDPWR
- removed copper zone on F.Cu, net GNDPWR
Other:
- board size 91.6 x 56.5 mm -> 318 x 127 mm
