File: Hardware/feng.sch (KiCad schematic (older format))
At the start: 220 parts, among them SW1 SW_SPST, SW10 SW_SPST, SW11 SW_SPST, SW12 SW_SPST, SW13 SW_SPST, SW14 SW_SPST, SW15 SW_SPST, SW16 SW_SPST, SW17 SW_SPST, SW18 SW_SPST, SW19 SW_SPST, SW2 SW_SPST, SW20 SW_SPST, SW21 SW_SPST, SW22 SW_SPST, SW23 SW_SPST, SW24 SW_SPST, SW3 SW_SPST, SW4 SW_SPST, SW5 SW_SPST, SW6 SW_SPST, SW7 SW_SPST, SW8 SW_SPST, SW9 SW_SPST, U1 74HC165D, U2 74HC165D, U3 74HC165D

Commit message: pcb_50%
Parts:
- C1, C3, C4, C5, C6, C7: renamed from C?; footprint (none) -> Capacitors:0805
- C2, C8: renamed from C?; value 20pf -> 22pf; footprint (none) -> Capacitors:0805
- D1, D10, D11, D12, D13, D14, D15, D16, D17, D18, D19, D2, D20, D21, D22, D23, D24, D25, D26, D27, D28, D29, D3, D30, D31, D32, D33, D34, D35, D36, D37, D38, D39, D4, D40, D41, D42, D43, D44, D45, D46, D47, D48, D49, D5, D50, D51, D52, D53, D54, D55, D56, D57, D58, D59, D6, D60, D61, D62, D63, D64, D65, D66, D67, D68, D69, D7, D70, D71, D72, D73, D74, D75, D76, D77, D78, D79, D8, D80, D81, D82, D83, D84, D85, D9: renamed from D?; footprint LED_SMD:LED_WS2812B_PLCC4_5.0x5.0mm_P3.2mm -> Hardware:LED_WS2812B_PLCC4_5.0x5.0mm_P3.2mm
- J1: renamed from J?; footprint (none) -> Connector_PinHeader_2.54mm:PinHeader_1x04_P2.54mm_Vertical
- J2: renamed from J?; footprint (none) -> Connector_USB:USB_C_Receptacle_Palconn_UTC16-G
- R1, R2, R3, R4, R5, R6, R7: renamed from R?; footprint (none) -> Resistors:0805
- SW1, SW10, SW11, SW12, SW13, SW14, SW15, SW16, SW17, SW18, SW19, SW2, SW20, SW21, SW22, SW23, SW24, SW25, SW26, SW27, SW28, SW29, SW3, SW30, SW31, SW32, SW33, SW34, SW35, SW36, SW37, SW38, SW39, SW4, SW40, SW41, SW42, SW43, SW44, SW45, SW46, SW47, SW48, SW49, SW5, SW50, SW51, SW52, SW53, SW54, SW55, SW56, SW6, SW7, SW8, SW81, SW82, SW9: renamed from SW?; footprint Button_Switch_THT:SW_DIP_SPSTx01_Slide_6.7x4.1mm_W7.62mm_P2.54mm_LowProfile -> Switch_Keyboard_Hotswap_Kailh:SW_Hotswap_Kailh_MX_1.00u
- SW57: renamed from SW1; footprint Button_Switch_THT:SW_DIP_SPSTx01_Slide_6.7x4.1mm_W7.62mm_P2.54mm_LowProfile -> Switch_Keyboard_Hotswap_Kailh:SW_Hotswap_Kailh_MX_1.00u
- SW58: renamed from SW2; footprint Button_Switch_THT:SW_DIP_SPSTx01_Slide_6.7x4.1mm_W7.62mm_P2.54mm_LowProfile -> Switch_Keyboard_Hotswap_Kailh:SW_Hotswap_Kailh_MX_1.00u
- SW59: renamed from SW3; footprint Button_Switch_THT:SW_DIP_SPSTx01_Slide_6.7x4.1mm_W7.62mm_P2.54mm_LowProfile -> Switch_Keyboard_Hotswap_Kailh:SW_Hotswap_Kailh_MX_1.00u
- SW60: renamed from SW4; footprint Button_Switch_THT:SW_DIP_SPSTx01_Slide_6.7x4.1mm_W7.62mm_P2.54mm_LowProfile -> Switch_Keyboard_Hotswap_Kailh:SW_Hotswap_Kailh_MX_1.00u
- SW61: renamed from SW5; footprint Button_Switch_THT:SW_DIP_SPSTx01_Slide_6.7x4.1mm_W7.62mm_P2.54mm_LowProfile -> Switch_Keyboard_Hotswap_Kailh:SW_Hotswap_Kailh_MX_1.00u
- SW62: renamed from SW6; footprint Button_Switch_THT:SW_DIP_SPSTx01_Slide_6.7x4.1mm_W7.62mm_P2.54mm_LowProfile -> Switch_Keyboard_Hotswap_Kailh:SW_Hotswap_Kailh_MX_1.00u
- SW63: renamed from SW7; footprint Button_Switch_THT:SW_DIP_SPSTx01_Slide_6.7x4.1mm_W7.62mm_P2.54mm_LowProfile -> Switch_Keyboard_Hotswap_Kailh:SW_Hotswap_Kailh_MX_1.00u
- SW64: renamed from SW8; footprint Button_Switch_THT:SW_DIP_SPSTx01_Slide_6.7x4.1mm_W7.62mm_P2.54mm_LowProfile -> Switch_Keyboard_Hotswap_Kailh:SW_Hotswap_Kailh_MX_1.00u
- SW65: renamed from SW9; footprint Button_Switch_THT:SW_DIP_SPSTx01_Slide_6.7x4.1mm_W7.62mm_P2.54mm_LowProfile -> Switch_Keyboard_Hotswap_Kailh:SW_Hotswap_Kailh_MX_1.00u
- SW66: renamed from SW10; footprint Button_Switch_THT:SW_DIP_SPSTx01_Slide_6.7x4.1mm_W7.62mm_P2.54mm_LowProfile -> Switch_Keyboard_Hotswap_Kailh:SW_Hotswap_Kailh_MX_1.00u
- SW67: renamed from SW11; footprint Button_Switch_THT:SW_DIP_SPSTx01_Slide_6.7x4.1mm_W7.62mm_P2.54mm_LowProfile -> Switch_Keyboard_Hotswap_Kailh:SW_Hotswap_Kailh_MX_1.00u
- SW68: renamed from SW12; footprint Button_Switch_THT:SW_DIP_SPSTx01_Slide_6.7x4.1mm_W7.62mm_P2.54mm_LowProfile -> Switch_Keyboard_Hotswap_Kailh:SW_Hotswap_Kailh_MX_1.00u
- SW69: renamed from SW13; footprint Button_Switch_THT:SW_DIP_SPSTx01_Slide_6.7x4.1mm_W7.62mm_P2.54mm_LowProfile -> Switch_Keyboard_Hotswap_Kailh:SW_Hotswap_Kailh_MX_1.00u
- SW70: renamed from SW14; footprint Button_Switch_THT:SW_DIP_SPSTx01_Slide_6.7x4.1mm_W7.62mm_P2.54mm_LowProfile -> Switch_Keyboard_Hotswap_Kailh:SW_Hotswap_Kailh_MX_1.00u
- SW71: renamed from SW15; footprint Button_Switch_THT:SW_DIP_SPSTx01_Slide_6.7x4.1mm_W7.62mm_P2.54mm_LowProfile -> Switch_Keyboard_Hotswap_Kailh:SW_Hotswap_Kailh_MX_1.00u
- SW72: renamed from SW16; footprint Button_Switch_THT:SW_DIP_SPSTx01_Slide_6.7x4.1mm_W7.62mm_P2.54mm_LowProfile -> Switch_Keyboard_Hotswap_Kailh:SW_Hotswap_Kailh_MX_1.00u
- SW73: renamed from SW17; footprint Button_Switch_THT:SW_DIP_SPSTx01_Slide_6.7x4.1mm_W7.62mm_P2.54mm_LowProfile -> Switch_Keyboard_Hotswap_Kailh:SW_Hotswap_Kailh_MX_1.00u
- SW74: renamed from SW18; footprint Button_Switch_THT:SW_DIP_SPSTx01_Slide_6.7x4.1mm_W7.62mm_P2.54mm_LowProfile -> Switch_Keyboard_Hotswap_Kailh:SW_Hotswap_Kailh_MX_1.00u
- SW75: renamed from SW19; footprint Button_Switch_THT:SW_DIP_SPSTx01_Slide_6.7x4.1mm_W7.62mm_P2.54mm_LowProfile -> Switch_Keyboard_Hotswap_Kailh:SW_Hotswap_Kailh_MX_1.00u
- SW76: renamed from SW20; footprint Button_Switch_THT:SW_DIP_SPSTx01_Slide_6.7x4.1mm_W7.62mm_P2.54mm_LowProfile -> Switch_Keyboard_Hotswap_Kailh:SW_Hotswap_Kailh_MX_1.00u
- SW77: renamed from SW21; footprint Button_Switch_THT:SW_DIP_SPSTx01_Slide_6.7x4.1mm_W7.62mm_P2.54mm_LowProfile -> Switch_Keyboard_Hotswap_Kailh:SW_Hotswap_Kailh_MX_1.00u
- SW78: renamed from SW22; footprint Button_Switch_THT:SW_DIP_SPSTx01_Slide_6.7x4.1mm_W7.62mm_P2.54mm_LowProfile -> Switch_Keyboard_Hotswap_Kailh:SW_Hotswap_Kailh_MX_1.00u
- SW79: renamed from SW23; footprint Button_Switch_THT:SW_DIP_SPSTx01_Slide_6.7x4.1mm_W7.62mm_P2.54mm_LowProfile -> Switch_Keyboard_Hotswap_Kailh:SW_Hotswap_Kailh_MX_1.00u
- SW80: renamed from SW24; footprint Button_Switch_THT:SW_DIP_SPSTx01_Slide_6.7x4.1mm_W7.62mm_P2.54mm_LowProfile -> Switch_Keyboard_Hotswap_Kailh:SW_Hotswap_Kailh_MX_1.00u
- SW83: renamed from SW?; footprint (none) -> Hardware:keyboard-RotaryEncoder_Alps_EC12E-Switch_Vertical_H20mm_CircularMountingHoles
- Y1: renamed from Y?; footprint (none) -> Crystal:Crystal_HC49-4H_Vertical
- gave numbers to parts that had none: 25
- renumbered RN3 to RN10, RN4 to RN19, RN5 to RN20, RN6 to RN21, RN1 to RN8, RN2 to RN9, U3 to U10, U1 to U8, U2 to U9
Other:
- moved on the sheet: R2, Y1

Commit message: pcb done
Parts:
- removed D83, D84, D85: WS2812B, Hardware:LED_WS2812B_PLCC4_5.0x5.0mm_P3.2mm, symbol LED:WS2812B
- added D86: LED, LED_SMD:LED_0805_2012Metric, symbol Device:LED
- added R8: 1K, Resistors:0805, symbol Device:R_Small
- D1, D10, D11, D12, D13, D14, D15, D16, D17, D18, D19, D2, D20, D21, D22, D23, D24, D25, D26, D27, D28, D29, D3, D30, D31, D32, D33, D34, D35, D36, D37, D38, D39, D4, D40, D41, D42, D43, D44, D45, D46, D47, D48, D49, D5, D50, D51, D52, D53, D54, D55, D56, D57, D58, D59, D6, D60, D61, D62, D63, D64, D65, D66, D67, D68, D69, D7, D70, D71, D72, D73, D74, D75, D76, D77, D78, D79, D8, D80, D81, D82, D9: footprint Hardware:LED_WS2812B_PLCC4_5.0x5.0mm_P3.2mm -> Switch_Keyboard_Alps_Matias:LED_WS2812B_PLCC4_5.0x5.0mm_P3.2mm
Connections:
- net GNDPWR: now also D86.1 (K)
- net CAPS_LED: now reaches U12.27 (PB14)
- net CAPS_LED: now also R8.2
- new net: D86.2 (A), R8.1
- no-connect marks 40 -> 42

Commit message: patch for c6 chip and change some code
Parts:
- added C10, C12: 0.1uf, Capacitors:0805, symbol Device:C_Small
- added C11, C9: 10uf, Capacitors:0805, symbol Device:C_Small
- added D83: LED, LED_SMD:LED_0805_2012Metric, symbol Device:LED
- added R9: 1K, Resistors:0805, symbol Device:R_Small
- added U13: AMS1117-3.3, Package_TO_SOT_SMD:SOT-223-3_TabPin2, symbol Regulator_Linear:AMS1117-3.3
Connections:
- net +3V3: now also C11.2, C12.2, R9.2, U13.2 (VO); no longer J2.A4 (VBUS), J2.A9 (VBUS), J2.B4 (VBUS), J2.B9 (VBUS)
- net GNDPWR: now also C10.1, C11.1, C12.1, C9.1, D83.1 (K), U13.1 (GND)
- new net: D83.2 (A), R9.1
- new net +5V: C10.2, C9.2, J2.A4 (VBUS), J2.A9 (VBUS), J2.B4 (VBUS), J2.B9 (VBUS), U13.3 (VI)
Changed lines of the file:
@@
 L power:+3.3V #PWR0198
 U 1 1 66508737
-P 8000 10250
-F 0 "#PWR0198" H 8000 10100 50  0001 C CNN
-F 1 "+3.3V" H 8015 10423 50  0000 C CNN
-F 2 "" H 8000 10250 50  0001 C CNN
-F 3 "" H 8000 10250 50  0001 C CNN
-	1    8000 10250
+P 10250 11450
+F 0 "#PWR0198" H 10250 11300 50  0001 C CNN
+F 1 "+3.3V" H 10265 11623 50  0000 C CNN
+F 2 "" H 10250 11450 50  0001 C CNN
+F 3 "" H 10250 11450 50  0001 C CNN
+	1    10250 11450
 	1    0    0    -1
 $EndComp
@@
 Wire Notes Line
 	9900 13300 9900 9000
-Wire Notes Line
-	550  13300 9900 13300
 $Comp
 L Connector_Generic:Conn_01x04 J1
@@
 Wire Notes Line
 	9900 11200 12100 11200
-Wire Notes Line
-	12100 8950 12100 11200
 $Comp
 L Device:R_Small R8
@@
 NoConn ~ 22050 3550
 NoConn ~ 22150 3550
+Wire Notes Line
+	9900 12050 12100 12050
+$Comp
+L Device:R_Small R9
+U 1 1 632EBD99
+P 10750 11450
+F 0 "R9" V 10800 11300 50  0000 C CNN
+F 1 "1K" V 10850 11450 50  0000 C CNN
+F 2 "Resistors:0805" H 10750 11450 50  0001 C CNN
+F 3 "~" H 10750 11450 50  0001 C CNN
+	1    10750 11450
+	0    1    1    0
+$EndComp
+$Comp
+L Device:LED D83
+U 1 1 632EBD9F
+P 11300 11600
+F 0 "D83" V 11339 11482 50  0000 R CNN
+F 1 "LED" V 11248 11482 50  0000 R CNN
+F 2 "LED_SMD:LED_0805_2012Metric" H 11300 11600 50  0001 C CNN
+F 3 "~" H 11300 11600 50  0001 C CNN
+	1    11300 11600
+	0    -1   -1   0
+$EndComp
+$Comp
+L power:GNDPWR #PWR0177
+U 1 1 632EBDA5
+P 11300 11850
+F 0 "#PWR0177" H 11300 11650 50  0001 C CNN
+F 1 "GNDPWR" H 11304 11696 50  0000 C CNN
+F 2 "Connector_PinHeader_2.54mm:PinHeader_1x01_P2.54mm_Vertical" H 11300 11800 50  0001 C CNN
+F 3 "" H 11300 11800 50  0001 C CNN
+	1    11300 11850
+	1    0    0    -1
+$EndComp
+Wire Wire Line
+	10850 11450 11300 11450
+Wire Wire Line
+	11300 11750 11300 11850
+Wire Wire Line
+	10250 11450 10650 11450
+$Comp
+L Device:C_Small C11
+U 1 1 6349C5D2
+P 11550 12650
+F 0 "C11" H 11458 12604 50  0000 R CNN
+F 1 "10uf" H 11458 12695 50  0000 R CNN
+F 2 "Capacitors:0805" H 11550 12650 50  0001 C CNN
+F 3 "~" H 11550 12650 50  0001 C CNN
+	1    11550 12650
+	-1   0    0    1
+$EndComp
+$Comp
+L Device:C_Small C10
+U 1 1 6349C5D8
+P 10800 12650
+F 0 "C10" H 10708 12604 50  0000 R CNN
+F 1 "0.1uf" H 10708 12695 50  0000 R CNN
+F 2 "Capacitors:0805" H 10800 12650 50  0001 C CNN
+F 3 "~" H 10800 12650 50  0001 C CNN
+	1    10800 12650
+	-1   0    0    1
+$EndComp
+$Comp
+L Device:C_Small C12
+U 1 1 6349C5DE
+P 11800 12650
+F 0 "C12" H 11708 12604 50  0000 R CNN
+F 1 "0.1uf" H 11708 12695 50  0000 R CNN
+F 2 "Capacitors:0805" H 11800 12650 50  0001 C CNN
+F 3 "~" H 11800 12650 50  0001 C CNN
+	1    11800 12650
+	-1   0    0    1
+$EndComp
+$Comp
+L Device:C_Small C9
+U 1 1 6349C5E4
+P 10550 12650
+F 0 "C9" H 10458 12604 50  0000 R CNN
+F 1 "10uf" H 10458 12695 50  0000 R CNN
+F 2 "Capacitors:0805" H 10550 12650 50  0001 C CNN
+F 3 "~" H 10550 12650 50  0001 C CNN
+	1    10550 12650
+	-1   0    0    1
+$EndComp
+$Comp
+L Regulator_Linear:AMS1117-3.3 U13
+U 1 1 636DACD2
+P 11250 12550
+F 0 "U13" H 11250 12792 50  0000 C CNN
+F 1 "AMS1117-3.3" H 11250 12701 50  0000 C CNN
+F 2 "Package_TO_SOT_SMD:SOT-223-3_TabPin2" H 11250 12750 50  0001 C CNN
+F 3 "http://www.advanced-monolithic.com/pdf/ds1117.pdf" H 11350 12300 50  0001 C CNN
+	1    11250 12550
+	1    0    0    -1
+$EndComp
+$Comp
+L power:+3.3V #PWR0178
+U 1 1 636DD030
+P 11800 12550
+F 0 "#PWR0178" H 11800 12400 50  0001 C CNN
+F 1 "+3.3V" H 11815 12723 50  0000 C CNN
+F 2 "" H 11800 12550 50  0001 C CNN
+F 3 "" H 11800 12550 50  0001 C CNN
+	1    11800 12550
+	1    0    0    -1
+$EndComp
+Wire Wire Line
+	11550 12550 11800 12550
+Connection ~ 11550 12550
+Connection ~ 11800 12550
+Wire Wire Line
+	11800 12750 11550 12750
+Wire Wire Line
+	11550 12750 11550 12850
+Wire Wire Line
+	11550 12850 11250 12850
+Connection ~ 11550 12750
+Wire Wire Line
+	10550 12750 10800 12750
+Wire Wire Line
+	10800 12750 10800 12850
+Wire Wire Line
+	10800 12850 11250 12850
+Connection ~ 10800 12750
+Connection ~ 11250 12850
+Wire Wire Line
+	10950 12550 10800 12550
+Connection ~ 10800 12550
+Wire Wire Line
+	10800 12550 10550 12550
+$Comp
+L power:+5V #PWR0179
+U 1 1 63A4B2A7
+P 10550 12550
+F 0 "#PWR0179" H 10550 12400 50  0001 C CNN
+F 1 "+5V" H 10565 12723 50  0000 C CNN
+F 2 "" H 10550 12550 50  0001 C CNN
+F 3 "" H 10550 12550 50  0001 C CNN
+	1    10550 12550
+	1    0    0    -1
+$EndComp
+Connection ~ 10550 12550
+$Comp
+L power:+5V #PWR0190
+U 1 1 63A4B627
+P 8000 10250
+F 0 "#PWR0190" H 8000 10100 50  0001 C CNN
+F 1 "+5V" H 8015 10423 50  0000 C CNN
+F 2 "" H 8000 10250 50  0001 C CNN
+F 3 "" H 8000 10250 50  0001 C CNN
+	1    8000 10250
+	1    0    0    -1
+$EndComp
+Wire Notes Line
+	550  13300 12100 13300
+Wire Notes Line
+	12100 9000 12100 13300
+$Comp
+L power:GNDPWR #PWR?
+U 1 1 63425C9A
+P 11250 12850
+F 0 "#PWR?" H 11250 12650 50  0001 C CNN
+F 1 "GNDPWR" H 11254 12696 50  0000 C CNN
+F 2 "Connector_PinHeader_2.54mm:PinHeader_1x01_P2.54mm_Vertical" H 11250 12800 50  0001 C CNN
+F 3 "" H 11250 12800 50  0001 C CNN
+	1    11250 12850
+	1    0    0    -1
+$EndComp
 $EndSCHEMATC
